File: kicad/sensor-node.sch (KiCad schematic (older format))
At the start: 7 parts

Commit message: added basic wiring for the MCU and the radio
Parts:
- added C1: C, symbol C
- added C3, C?: 1µF, symbol C
- added C? (x4): 0.1µF, symbol C
- added C? (x3): 10µF, symbol C
- added C? (x2): 10nF, symbol C
- added D1: LED, symbol LED
- L1: renamed from L?; value 220 nH -> 220nH
- gave numbers to parts that had none: 6
Connections:
- net labels added: +3V3, SCL, SDA, S_ENABLE, S_INT
- net labels removed: VDD
- wire segments 18 -> 54
- no-connect marks 0 -> 38

Commit message: added sensor
Parts:
- added SBA1: Si7021-BA, symbol Si7021-BA
- gave numbers to parts that had none: 10
Connections:
- net labels added: RAD_ENABLE, RAD_INT, ~SEN_ENABLE
- net labels removed: S_ENABLE, S_INT
- no-connect marks 38 -> 39
Changed lines of the file:
@@
 SCL
 Text Label 10550 3700 0    60   ~ 0
-S_ENABLE
+RAD_ENABLE
 Text Label 10550 3800 0    60   ~ 0
-S_INT
+RAD_INT
 Text Label 4400 3150 2    60   ~ 0
 SDA
@@
 $EndComp
 $Comp
-L C C?
+L C C12
 U 1 1 58793969
 P 6800 4100
-F 0 "C?" H 6825 4200 50  0000 L CNN
+F 0 "C12" H 6825 4200 50  0000 L CNN
 F 1 "0.1µF" H 6825 4000 50  0000 L CNN
 F 2 "" H 6838 3950 50  0000 C CNN
@@
 $EndComp
 $Comp
-L C C?
+L C C13
 U 1 1 587939B0
 P 7100 4100
-F 0 "C?" H 7125 4200 50  0000 L CNN
+F 0 "C13" H 7125 4200 50  0000 L CNN
 F 1 "10µF" H 7125 4000 50  0000 L CNN
 F 2 "" H 7138 3950 50  0000 C CNN
@@
 $EndComp
 $Comp
-L GND #PWR?
+L GND #PWR010
 U 1 1 587939DD
 P 7100 4400
-F 0 "#PWR?" H 7100 4150 50  0001 C CNN
+F 0 "#PWR010" H 7100 4150 50  0001 C CNN
 F 1 "GND" H 7100 4250 50  0000 C CNN
 F 2 "" H 7100 4400 50  0000 C CNN
@@
 $EndComp
 $Comp
-L +3V3 #PWR?
+L +3V3 #PWR011
 U 1 1 58793A09
 P 7350 3950
-F 0 "#PWR?" H 7350 3800 50  0001 C CNN
+F 0 "#PWR011" H 7350 3800 50  0001 C CNN
 F 1 "+3V3" H 7350 4090 50  0000 C CNN
 F 2 "" H 7350 3950 50  0000 C CNN
@@
 	7100 4250 7100 4400
 $Comp
-L C C?
+L C C11
 U 1 1 58793B7A
 P 6800 3650
-F 0 "C?" H 6825 3750 50  0000 L CNN
+F 0 "C11" H 6825 3750 50  0000 L CNN
 F 1 "1µF" H 6825 3550 50  0000 L CNN
 F 2 "" H 6838 3500 50  0000 C CNN
@@
 $EndComp
 $Comp
-L GND #PWR?
+L GND #PWR012
 U 1 1 58793BA9
 P 6800 3400
-F 0 "#PWR?" H 6800 3150 50  0001 C CNN
+F 0 "#PWR012" H 6800 3150 50  0001 C CNN
 F 1 "GND" H 6800 3250 50  0000 C CNN
 F 2 "" H 6800 3400 50  0000 C CNN
@@
 	6800 3500 6800 3400
 $Comp
-L GND #PWR?
+L GND #PWR013
 U 1 1 58793D7C
 P 5350 4700
-F 0 "#PWR?" H 5350 4450 50  0001 C CNN
+F 0 "#PWR013" H 5350 4450 50  0001 C CNN
 F 1 "GND" H 5350 4550 50  0000 C CNN
 F 2 "" H 5350 4700 50  0000 C CNN
@@
 $EndComp
 $Comp
-L GND #PWR?
+L GND #PWR014
 U 1 1 58793DAA
 P 5850 5250
-F 0 "#PWR?" H 5850 5000 50  0001 C CNN
+F 0 "#PWR014" H 5850 5000 50  0001 C CNN
 F 1 "GND" H 5850 5100 50  0000 C CNN
 F 2 "" H 5850 5250 50  0000 C CNN
@@
 $EndComp
 $Comp
-L C C?
+L C C9
 U 1 1 58793DD8
 P 5850 5000
-F 0 "C?" H 5875 5100 50  0000 L CNN
+F 0 "C9" H 5875 5100 50  0000 L CNN
 F 1 "10nF" H 5875 4900 50  0000 L CNN
 F 2 "" H 5888 4850 50  0000 C CNN
@@
 $EndComp
 $Comp
-L C C?
+L C C7
 U 1 1 58793E0D
 P 5450 5000
-F 0 "C?" H 5475 5100 50  0000 L CNN
+F 0 "C7" H 5475 5100 50  0000 L CNN
 F 1 "10nF" H 5475 4900 50  0000 L CNN
 F 2 "" H 5488 4850 50  0000 C CNN
@@
 $EndComp
 $Comp
-L C C?
+L C C10
 U 1 1 58793E48
 P 6250 5000
-F 0 "C?" H 6275 5100 50  0000 L CNN
+F 0 "C10" H 6275 5100 50  0000 L CNN
 F 1 "10µF" H 6275 4900 50  0000 L CNN
 F 2 "" H 6288 4850 50  0000 C CNN
@@
 $EndComp
 $Comp
-L GND #PWR?
+L GND #PWR015
 U 1 1 58793F0E
 P 5450 5250
-F 0 "#PWR?" H 5450 5000 50  0001 C CNN
+F 0 "#PWR015" H 5450 5000 50  0001 C CNN
 F 1 "GND" H 5450 5100 50  0000 C CNN
 F 2 "" H 5450 5250 50  0000 C CNN
@@
 $EndComp
 $Comp
-L +3V3 #PWR?
+L +3V3 #PWR016
 U 1 1 58793F42
 P 6500 4850
-F 0 "#PWR?" H 6500 4700 50  0001 C CNN
+F 0 "#PWR016" H 6500 4700 50  0001 C CNN
 F 1 "+3V3" H 6500 4990 50  0000 C CNN
 F 2 "" H 6500 4850 50  0000 C CNN
@@
 	0    1    1    0
 $EndComp
-Wire Wire Line
-	5450 4700 5450 4850
-Wire Wire Line
-	5450 4850 6500 4850
 Connection ~ 5850 4850
 Connection ~ 6250 4850
@@
 	5850 5150 6250 5150
 $Comp
-L GND #PWR?
+L GND #PWR017
 U 1 1 587942FF
 P 4400 3550
-F 0 "#PWR?" H 4400 3300 50  0001 C CNN
+F 0 "#PWR017" H 4400 3300 50  0001 C CNN
 F 1 "GND" H 4400 3400 50  0000 C CNN
 F 2 "" H 4400 3550 50  0000 C CNN
@@
 $EndComp
 $Comp
-L C C?
+L C C8
 U 1 1 58794495
 P 5650 5350
-F 0 "C?" H 5675 5450 50  0000 L CNN
+F 0 "C8" H 5675 5450 50  0000 L CNN
 F 1 "0.1µF" H 5675 5250 50  0000 L CNN
 F 2 "" H 5688 5200 50  0000 C CNN
@@
 $EndComp
 $Comp
-L GND #PWR?
+L GND #PWR018
 U 1 1 58794543
 P 5650 5600
-F 0 "#PWR?" H 5650 5350 50  0001 C CNN
+F 0 "#PWR018" H 5650 5350 50  0001 C CNN
 F 1 "GND" H 5650 5450 50  0000 C CNN
 F 2 "" H 5650 5600 50  0000 C CNN
@@
 	5750 5150 5750 4700
 $Comp
-L C C?
+L C C4
 U 1 1 5879D002
 P 4050 3450
-F 0 "C?" H 4075 3550 50  0000 L CNN
+F 0 "C4" H 4075 3550 50  0000 L CNN
 F 1 "0.1µF" H 4075 3350 50  0000 L CNN
 F 2 "" H 4088 3300 50  0000 C CNN
@@
 $EndComp
 $Comp
-L C C?
+L C C6
 U 1 1 5879D061
 P 5350 2400
-F 0 "C?" H 5375 2500 50  0000 L CNN
+F 0 "C6" H 5375 2500 50  0000 L CNN
 F 1 "0.1µF" H 5375 2300 50  0000 L CNN
 F 2 "" H 5388 2250 50  0000 C CNN
@@
 $EndComp
 $Comp
-L C C?
+L C C5
 U 1 1 5879D0E8
 P 5100 5350
-F 0 "C?" H 5125 5450 50  0000 L CNN
+F 0 "C5" H 5125 5450 50  0000 L CNN
 F 1 "10µF" H 5125 5250 50  0000 L CNN
 F 2 "" H 5138 5200 50  0000 C CNN
@@
 	5100 5200 5100 5150
 $Comp
-L GND #PWR?
+L GND #PWR019
 U 1 1 5879D519
 P 5100 5600
-F 0 "#PWR?" H 5100 5350 50  0001 C CNN
+F 0 "#PWR019" H 5100 5350 50  0001 C CNN
 F 1 "GND" H 5100 5450 50  0000 C CNN
 F 2 "" H 5100 5600 50  0000 C CNN
@@
 $EndComp
 $Comp
-L GND #PWR?
+L GND #PWR020
 U 1 1 5879D5A5
 P 3800 3450
-F 0 "#PWR?" H 3800 3200 50  0001 C CNN
+F 0 "#PWR020" H 3800 3200 50  0001 C CNN
 F 1 "GND" H 3800 3300 50  0000 C CNN
 F 2 "" H 3800 3450 50  0000 C CNN
@@
 $EndComp
 $Comp
-L GND #PWR?
+L GND #PWR021
 U 1 1 5879D609
 P 5350 2150
-F 0 "#PWR?" H 5350 1900 50  0001 C CNN
+F 0 "#PWR021" H 5350 1900 50  0001 C CNN
 F 1 "GND" H 5350 2000 50  0000 C CNN
 F 2 "" H 5350 2150 50  0000 C CNN
@@
 	5100 5500 5100 5600
 $Comp
-L +3V3 #PWR?
+L +3V3 #PWR022
 U 1 1 5879D7EB
 P 4200 5150
-F 0 "#PWR?" H 4200 5000 50  0001 C CNN
+F 0 "#PWR022" H 4200 5000 50  0001 C CNN
 F 1 "+3V3" H 4200 5290 50  0000 C CNN
 F 2 "" H 4200 5150 50  0000 C CNN
@@
 	0    -1   -1   0
 $EndComp
+$Comp
+L Si7021-BA SBA1
+U 1 1 5879DD92
+P 2250 5350
+F 0 "SBA1" H 2500 5000 60  0000 C CNN
+F 1 "Si7021-BA" H 2100 5350 60  0000 C CNN
+F 2 "" H 2150 5400 60  0001 C CNN
+F 3 "" H 2150 5400 60  0001 C CNN
+	1    2250 5350
+	1    0    0    -1
+$EndComp
+Text Label 2800 5150 0    60   ~ 0
+SDA
+Text Label 2800 5250 0    60   ~ 0
+SCL
+NoConn ~ 2800 5450
+$Comp
+L +3V3 #PWR023
+U 1 1 5879DF12
+P 2800 5550
+F 0 "#PWR023" H 2800 5400 50  0001 C CNN
+F 1 "+3V3" H 2800 5690 50  0000 C CNN
+F 2 "" H 2800 5550 50  0000 C CNN
+F 3 "" H 2800 5550 50  0000 C CNN
+	1    2800 5550
+	0    1    1    0
+$EndComp
+Text Label 2800 5350 0    60   ~ 0
+~SEN_ENABLE
+Wire Wire Line
+	5450 4850 5450 4700
+Wire Wire Line
+	5450 4850 6500 4850
 $EndSCHEMATC

Commit message: updated pull-up values in the diagram
Parts:
- R1, R2: value R -> 10k
Changed lines of the file:
@@
 P 2900 3550
 F 0 "R1" V 2980 3550 50  0000 C CNN
-F 1 "R" V 2900 3550 50  0000 C CNN
+F 1 "10k" V 2900 3550 50  0000 C CNN
 F 2 "" V 2830 3550 50  0000 C CNN
 F 3 "" H 2900 3550 50  0000 C CNN
@@
 P 3100 3650
 F 0 "R2" V 3180 3650 50  0000 C CNN
-F 1 "R" V 3100 3650 50  0000 C CNN
+F 1 "10k" V 3100 3650 50  0000 C CNN
 F 2 "" V 3030 3650 50  0000 C CNN
 F 3 "" H 3100 3650 50  0000 C CNN

Commit message: added debug connector
Parts:
- added CD?: CortexDebug, symbol CortexDebug
Connections:
- net labels added: SWCLK, SWDIO, SWO, ~RESET
- wire segments 54 -> 60
- no-connect marks 39 -> 35
Changed lines of the file:
@@
 NoConn ~ 5550 2700
 NoConn ~ 5650 2700
-NoConn ~ 5750 2700
-NoConn ~ 5850 2700
-NoConn ~ 5950 2700
 NoConn ~ 6400 3150
 NoConn ~ 6400 3250
@@
 NoConn ~ 5550 4700
 NoConn ~ 5250 4700
-NoConn ~ 5150 4700
 NoConn ~ 5050 4700
 NoConn ~ 4950 4700
@@
 Wire Wire Line
 	5450 4850 6500 4850
+$Comp
+L CortexDebug CD?
+U 1 1 58832D91
+P 2300 6550
+F 0 "CD?" H 2800 6200 60  0000 C CNN
+F 1 "CortexDebug" H 2300 6550 60  0000 C CNN
+F 2 "" H 2600 6450 60  0001 C CNN
+F 3 "" H 2600 6450 60  0001 C CNN
+	1    2300 6550
+	1    0    0    -1
+$EndComp
+Text Label 5950 2700 1    60   ~ 0
+SWCLK
+Text Label 5850 2700 1    60   ~ 0
+SWDIO
+Text Label 5750 2700 1    60   ~ 0
+SWO
+Text Label 3100 6350 0    60   ~ 0
+SWDIO
+Text Label 3100 6450 0    60   ~ 0
+SWCLK
+Text Label 3100 6550 0    60   ~ 0
+SWO
+Text Label 3100 6750 0    60   ~ 0
+~RESET
+$Comp
+L GND #PWR?
+U 1 1 58833835
+P 1400 6900
+F 0 "#PWR?" H 1400 6650 50  0001 C CNN
+F 1 "GND" H 1400 6750 50  0000 C CNN
+F 2 "" H 1400 6900 50  0000 C CNN
+F 3 "" H 1400 6900 50  0000 C CNN
+	1    1400 6900
+	1    0    0    -1
+$EndComp
+Wire Wire Line
+	1400 6450 1400 6900
+Wire Wire Line
+	1400 6750 1500 6750
+Wire Wire Line
+	1400 6550 1500 6550
+Connection ~ 1400 6750
+Wire Wire Line
+	1400 6450 1500 6450
+Connection ~ 1400 6550
+$Comp
+L +3V3 #PWR?
+U 1 1 58833AC8
+P 1400 6150
+F 0 "#PWR?" H 1400 6000 50  0001 C CNN
+F 1 "+3V3" H 1400 6290 50  0000 C CNN
+F 2 "" H 1400 6150 50  0000 C CNN
+F 3 "" H 1400 6150 50  0000 C CNN
+	1    1400 6150
+	1    0    0    -1
+$EndComp
+Wire Wire Line
+	1400 6150 1400 6350
+Wire Wire Line
+	1400 6350 1500 6350
+Text Label 5150 4700 3    60   ~ 0
+~RESET
 $EndSCHEMATC

Commit message: fixed some minor problems
Parts:
- gave numbers to parts that had none: 1
Connections:
- wire segments 60 -> 63
- no-connect marks 35 -> 34
Changed lines of the file:
@@
 NoConn ~ 5050 2700
 NoConn ~ 5150 2700
-NoConn ~ 5250 2700
 NoConn ~ 5450 2700
 NoConn ~ 5550 2700
@@
 	5450 4850 6500 4850
 $Comp
-L CortexDebug CD?
+L CortexDebug CD1
 U 1 1 58832D91
 P 2300 6550
-F 0 "CD?" H 2800 6200 60  0000 C CNN
+F 0 "CD1" H 2800 6200 60  0000 C CNN
 F 1 "CortexDebug" H 2300 6550 60  0000 C CNN
 F 2 "" H 2600 6450 60  0001 C CNN
@@
 ~RESET
 $Comp
-L GND #PWR?
+L GND #PWR024
 U 1 1 58833835
 P 1400 6900
-F 0 "#PWR?" H 1400 6650 50  0001 C CNN
+F 0 "#PWR024" H 1400 6650 50  0001 C CNN
 F 1 "GND" H 1400 6750 50  0000 C CNN
 F 2 "" H 1400 6900 50  0000 C CNN
@@
 Connection ~ 1400 6550
 $Comp
-L +3V3 #PWR?
+L +3V3 #PWR025
 U 1 1 58833AC8
 P 1400 6150
-F 0 "#PWR?" H 1400 6000 50  0001 C CNN
+F 0 "#PWR025" H 1400 6000 50  0001 C CNN
 F 1 "+3V3" H 1400 6290 50  0000 C CNN
 F 2 "" H 1400 6150 50  0000 C CNN
@@
 Text Label 5150 4700 3    60   ~ 0
 ~RESET
+$Comp
+L GND #PWR026
+U 1 1 58833543
+P 5150 2350
+F 0 "#PWR026" H 5150 2100 50  0001 C CNN
+F 1 "GND" H 5150 2200 50  0000 C CNN
+F 2 "" H 5150 2350 50  0000 C CNN
+F 3 "" H 5150 2350 50  0000 C CNN
+	1    5150 2350
+	-1   0    0    1
+$EndComp
+Wire Wire Line
+	5150 2350 5150 2500
+Wire Wire Line
+	5150 2500 5250 2500
+Wire Wire Line
+	5250 2500 5250 2700
 $EndSCHEMATC
