File: kicad/sensor-node.sch (KiCad schematic (older format))
At the start: 22 parts

Commit message: started board layout
Parts:
- added C14: 1pF, Capacitors_SMD:C_0805_HandSoldering, symbol C
- BT1: footprint (none) -> Pin_Headers:Pin_Header_Angled_1x02
- C1: value C -> 1pF; footprint (none) -> Capacitors_SMD:C_0805_HandSoldering
- C10, C11, C12, C13, C2, C3, C4, C5, C6, C7, C8, C9: footprint (none) -> Capacitors_SMD:C_0805_HandSoldering
- CD1: footprint (none) -> Pin_Headers:Pin_Header_Angled_2x05
- D1: footprint (none) -> LEDs:LED_0603
- EFM1: footprint (none) -> Housings_QFP:TQFP-48_7x7mm_Pitch0.5mm
- L1, R1, R2: footprint (none) -> Resistors_SMD:R_0805_HandSoldering
- S1: footprint (none) -> Housings_SSOP:MSOP-10_3x3mm_Pitch0.5mm
- SBA1: footprint (none) -> Pin_Headers:Pin_Header_Straight_1x05
Connections:
- wire segments 63 -> 65

Commit message: added custom footprints
Parts:
- BT1: footprint Pin_Headers:Pin_Header_Angled_1x02 -> sensor-node:HU2032-LF
- CD1: footprint Pin_Headers:Pin_Header_Angled_2x05 -> sensor-node:CORTEX-DEBUG-EDGE
Changed lines of the file:
@@
 F 0 "BT1" H 1200 3600 50  0000 L CNN
 F 1 "CR2032" H 1200 3500 50  0000 L CNN
-F 2 "Pin_Headers:Pin_Header_Angled_1x02" V 1100 3590 50  0001 C CNN
+F 2 "sensor-node:HU2032-LF" V 1100 3590 50  0001 C CNN
 F 3 "" V 1100 3590 50  0000 C CNN
 	1    1100 3550
@@
 F 0 "CD1" H 2800 6200 60  0000 C CNN
 F 1 "CortexDebug" H 2300 6550 60  0000 C CNN
-F 2 "Pin_Headers:Pin_Header_Angled_2x05" H 2600 6450 60  0001 C CNN
+F 2 "sensor-node:CORTEX-DEBUG-EDGE" H 2600 6450 60  0001 C CNN
 F 3 "" H 2600 6450 60  0001 C CNN
 	1    2300 6550

Commit message: automated bom creation and moved it to a separate page
Parts:
- BT1: value CR2032 -> CR2032Holder
Changed lines of the file:
@@
 P 1100 3550
 F 0 "BT1" H 1200 3600 50  0000 L CNN
-F 1 "CR2032" H 1200 3500 50  0000 L CNN
+F 1 "CR2032Holder" H 1200 3500 50  0000 L CNN
 F 2 "sensor-node:HU2032-LF" V 1100 3590 50  0001 C CNN
 F 3 "" V 1100 3590 50  0000 C CNN

Commit message: removed led
Parts:
- removed D1: LED, LEDs:LED_0603, symbol LED
Connections:
- wire segments 65 -> 62
- no-connect marks 34 -> 35
Changed lines of the file:
@@
-$EndComp
-$Comp
-L LED D1
-U 1 1 58792412
-P 10750 4300
-F 0 "D1" H 10750 4400 50  0000 C CNN
-F 1 "LED" H 10750 4200 50  0000 C CNN
-F 2 "LEDs:LED_0603" H 10750 4300 50  0001 C CNN
-F 3 "" H 10750 4300 50  0000 C CNN
-	1    10750 4300
-	0    1    1    0
 $EndComp
 $Comp
@@
 	1    9350 4150
 	1    0    0    -1
-$EndComp
-$Comp
-L +3V3 #PWR07
-U 1 1 58792727
-P 10750 4700
-F 0 "#PWR07" H 10750 4550 50  0001 C CNN
-F 1 "+3V3" H 10750 4840 50  0000 C CNN
-F 2 "" H 10750 4700 50  0000 C CNN
-F 3 "" H 10750 4700 50  0000 C CNN
-	1    10750 4700
-	-1   0    0    1
 $EndComp
 Text Label 10550 3500 0    60   ~ 0
@@
 Connection ~ 9050 4700
 Wire Wire Line
-	10750 4700 10750 4500
-Wire Wire Line
-	10750 4100 10750 3900
-Wire Wire Line
-	10750 3900 10550 3900
-Wire Wire Line
 	9300 3600 9350 3600
 Wire Wire Line
@@
 Wire Wire Line
 	7850 3900 8100 3900
+NoConn ~ 10550 3900
 $EndSCHEMATC

Commit message: added mounting holes and custom footprint for sensor module
Parts:
- SBA1: footprint Pin_Headers:Pin_Header_Straight_1x05 -> sensor-node:Si7021BA
Changed lines of the file:
@@
 SCL
 $Comp
-L +3V3 #PWR08
+L +3V3 #PWR07
 U 1 1 58792BC2
 P 2900 3950
-F 0 "#PWR08" H 2900 3800 50  0001 C CNN
+F 0 "#PWR07" H 2900 3800 50  0001 C CNN
 F 1 "+3V3" H 2900 4090 50  0000 C CNN
 F 2 "" H 2900 3950 50  0000 C CNN
@@
 NoConn ~ 4850 4700
 $Comp
-L GND #PWR09
+L GND #PWR08
 U 1 1 5879365E
 P 9350 4350
-F 0 "#PWR09" H 9350 4100 50  0001 C CNN
+F 0 "#PWR08" H 9350 4100 50  0001 C CNN
 F 1 "GND" H 9350 4200 50  0000 C CNN
 F 2 "" H 9350 4350 50  0000 C CNN
@@
 $EndComp
 $Comp
-L GND #PWR010
+L GND #PWR09
 U 1 1 587939DD
 P 7100 4400
-F 0 "#PWR010" H 7100 4150 50  0001 C CNN
+F 0 "#PWR09" H 7100 4150 50  0001 C CNN
 F 1 "GND" H 7100 4250 50  0000 C CNN
 F 2 "" H 7100 4400 50  0000 C CNN
@@
 $EndComp
 $Comp
-L +3V3 #PWR011
+L +3V3 #PWR010
 U 1 1 58793A09
 P 7350 3950
-F 0 "#PWR011" H 7350 3800 50  0001 C CNN
+F 0 "#PWR010" H 7350 3800 50  0001 C CNN
 F 1 "+3V3" H 7350 4090 50  0000 C CNN
 F 2 "" H 7350 3950 50  0000 C CNN
@@
 $EndComp
 $Comp
-L GND #PWR012
+L GND #PWR011
 U 1 1 58793BA9
 P 6800 3400
-F 0 "#PWR012" H 6800 3150 50  0001 C CNN
+F 0 "#PWR011" H 6800 3150 50  0001 C CNN
 F 1 "GND" H 6800 3250 50  0000 C CNN
 F 2 "" H 6800 3400 50  0000 C CNN
@@
 $EndComp
 $Comp
-L GND #PWR013
+L GND #PWR012
 U 1 1 58793D7C
 P 5350 4700
-F 0 "#PWR013" H 5350 4450 50  0001 C CNN
+F 0 "#PWR012" H 5350 4450 50  0001 C CNN
 F 1 "GND" H 5350 4550 50  0000 C CNN
 F 2 "" H 5350 4700 50  0000 C CNN
@@
 $EndComp
 $Comp
-L GND #PWR014
+L GND #PWR013
 U 1 1 58793DAA
 P 5850 5250
-F 0 "#PWR014" H 5850 5000 50  0001 C CNN
+F 0 "#PWR013" H 5850 5000 50  0001 C CNN
 F 1 "GND" H 5850 5100 50  0000 C CNN
 F 2 "" H 5850 5250 50  0000 C CNN
@@
 $EndComp
 $Comp
-L GND #PWR015
+L GND #PWR014
 U 1 1 58793F0E
 P 5450 5250
-F 0 "#PWR015" H 5450 5000 50  0001 C CNN
+F 0 "#PWR014" H 5450 5000 50  0001 C CNN
 F 1 "GND" H 5450 5100 50  0000 C CNN
 F 2 "" H 5450 5250 50  0000 C CNN
@@
 $EndComp
 $Comp
-L +3V3 #PWR016
+L +3V3 #PWR015
 U 1 1 58793F42
 P 6500 4850
-F 0 "#PWR016" H 6500 4700 50  0001 C CNN
+F 0 "#PWR015" H 6500 4700 50  0001 C CNN
 F 1 "+3V3" H 6500 4990 50  0000 C CNN
 F 2 "" H 6500 4850 50  0000 C CNN
@@
 $EndComp
 $Comp
-L GND #PWR017
+L GND #PWR016
 U 1 1 587942FF
 P 4400 3550
-F 0 "#PWR017" H 4400 3300 50  0001 C CNN
+F 0 "#PWR016" H 4400 3300 50  0001 C CNN
 F 1 "GND" H 4400 3400 50  0000 C CNN
 F 2 "" H 4400 3550 50  0000 C CNN
@@
 $EndComp
 $Comp
-L GND #PWR018
+L GND #PWR017
 U 1 1 58794543
 P 5650 5600
-F 0 "#PWR018" H 5650 5350 50  0001 C CNN
+F 0 "#PWR017" H 5650 5350 50  0001 C CNN
 F 1 "GND" H 5650 5450 50  0000 C CNN
 F 2 "" H 5650 5600 50  0000 C CNN
@@
 $EndComp
 $Comp
-L GND #PWR019
+L GND #PWR018
 U 1 1 5879D519
 P 5100 5600
-F 0 "#PWR019" H 5100 5350 50  0001 C CNN
+F 0 "#PWR018" H 5100 5350 50  0001 C CNN
 F 1 "GND" H 5100 5450 50  0000 C CNN
 F 2 "" H 5100 5600 50  0000 C CNN
@@
 $EndComp
 $Comp
-L GND #PWR020
+L GND #PWR019
 U 1 1 5879D5A5
 P 3800 3450
-F 0 "#PWR020" H 3800 3200 50  0001 C CNN
+F 0 "#PWR019" H 3800 3200 50  0001 C CNN
 F 1 "GND" H 3800 3300 50  0000 C CNN
 F 2 "" H 3800 3450 50  0000 C CNN
@@
 $EndComp
 $Comp
-L GND #PWR021
+L GND #PWR020
 U 1 1 5879D609
 P 5350 2150
-F 0 "#PWR021" H 5350 1900 50  0001 C CNN
+F 0 "#PWR020" H 5350 1900 50  0001 C CNN
 F 1 "GND" H 5350 2000 50  0000 C CNN
 F 2 "" H 5350 2150 50  0000 C CNN
@@
 $EndComp
 $Comp
-L +3V3 #PWR022
+L +3V3 #PWR021
 U 1 1 5879D7EB
 P 4200 5150
-F 0 "#PWR022" H 4200 5000 50  0001 C CNN
+F 0 "#PWR021" H 4200 5000 50  0001 C CNN
 F 1 "+3V3" H 4200 5290 50  0000 C CNN
 F 2 "" H 4200 5150 50  0000 C CNN
@@
 F 0 "SBA1" H 2500 5000 60  0000 C CNN
 F 1 "Si7021-BA" H 2100 5350 60  0000 C CNN
-F 2 "Pin_Headers:Pin_Header_Straight_1x05" H 2150 5400 60  0001 C CNN
+F 2 "sensor-node:Si7021BA" H 2150 5400 60  0001 C CNN
 F 3 "" H 2150 5400 60  0001 C CNN
 	1    2250 5350
@@
 NoConn ~ 2800 5450
 $Comp
-L +3V3 #PWR023
+L +3V3 #PWR022
 U 1 1 5879DF12
 P 2800 5550
-F 0 "#PWR023" H 2800 5400 50  0001 C CNN
+F 0 "#PWR022" H 2800 5400 50  0001 C CNN
 F 1 "+3V3" H 2800 5690 50  0000 C CNN
 F 2 "" H 2800 5550 50  0000 C CNN
@@
 ~RESET
 $Comp
-L GND #PWR024
+L GND #PWR023
 U 1 1 58833835
 P 1400 6900
-F 0 "#PWR024" H 1400 6650 50  0001 C CNN
+F 0 "#PWR023" H 1400 6650 50  0001 C CNN
 F 1 "GND" H 1400 6750 50  0000 C CNN
 F 2 "" H 1400 6900 50  0000 C CNN
@@
 $EndComp
 $Comp
-L +3V3 #PWR025
+L +3V3 #PWR024
 U 1 1 58833AC8
 P 1400 6150
-F 0 "#PWR025" H 1400 6000 50  0001 C CNN
+F 0 "#PWR024" H 1400 6000 50  0001 C CNN
 F 1 "+3V3" H 1400 6290 50  0000 C CNN
 F 2 "" H 1400 6150 50  0000 C CNN
@@
 ~RESET
 $Comp
-L GND #PWR026
+L GND #PWR025
 U 1 1 58833543
 P 5150 2350
-F 0 "#PWR026" H 5150 2100 50  0001 C CNN
+F 0 "#PWR025" H 5150 2100 50  0001 C CNN
 F 1 "GND" H 5150 2200 50  0000 C CNN
 F 2 "" H 5150 2350 50  0000 C CNN

Commit message: redrew antenna
Connections:
- no-connect marks 35 -> 32
Changed lines of the file:
@@
 Text Label 3450 3200 0    60   ~ 0
 SDA
-NoConn ~ 4850 2700
-NoConn ~ 4950 2700
-NoConn ~ 5050 2700
 NoConn ~ 5150 2700
 NoConn ~ 5450 2700
@@
 	7850 3900 8100 3900
 NoConn ~ 10550 3900
+Text Label 4950 2700 1    60   ~ 0
+RAD_INT
+Text Label 4850 2700 1    60   ~ 0
+RAD_ENABLE
+Text Label 5050 2700 1    60   ~ 0
+~SEN_ENABLE
 $EndSCHEMATC

Commit message: added a decoupling capacitor
Parts:
- added C15: 10µF, Capacitors_SMD:C_0805_HandSoldering, symbol C
Connections:
- wire segments 62 -> 64
Changed lines of the file:
@@
 L GND #PWR020
 U 1 1 5879D609
-P 5350 2150
-F 0 "#PWR020" H 5350 1900 50  0001 C CNN
-F 1 "GND" H 5350 2000 50  0000 C CNN
-F 2 "" H 5350 2150 50  0000 C CNN
-F 3 "" H 5350 2150 50  0000 C CNN
-	1    5350 2150
+P 5350 2100
+F 0 "#PWR020" H 5350 1850 50  0001 C CNN
+F 1 "GND" H 5350 1950 50  0000 C CNN
+F 2 "" H 5350 2100 50  0000 C CNN
+F 3 "" H 5350 2100 50  0000 C CNN
+	1    5350 2100
 	-1   0    0    1
 $EndComp
@@
 	5350 2550 5350 2700
 Wire Wire Line
-	5350 2600 4200 2600
+	4200 2600 5350 2600
 Wire Wire Line
 	4200 2600 4200 5150
@@
 	5100 5200 5100 5150
 Wire Wire Line
-	5350 2150 5350 2250
+	5350 2100 5350 2250
 Wire Wire Line
 	3900 3450 3800 3450
@@
 Text Label 5050 2700 1    60   ~ 0
 ~SEN_ENABLE
+$Comp
+L C C15
+U 1 1 589EE79E
+P 4500 2400
+F 0 "C15" H 4525 2500 50  0000 L CNN
+F 1 "10µF" H 4525 2300 50  0000 L CNN
+F 2 "Capacitors_SMD:C_0805_HandSoldering" H 4538 2250 50  0001 C CNN
+F 3 "" H 4500 2400 50  0000 C CNN
+	1    4500 2400
+	1    0    0    -1
+$EndComp
+$Comp
+L GND #PWR026
+U 1 1 589EE7EB
+P 4500 2100
+F 0 "#PWR026" H 4500 1850 50  0001 C CNN
+F 1 "GND" H 4500 1950 50  0000 C CNN
+F 2 "" H 4500 2100 50  0000 C CNN
+F 3 "" H 4500 2100 50  0000 C CNN
+	1    4500 2100
+	-1   0    0    1
+$EndComp
+Wire Wire Line
+	4500 2550 4500 2600
+Connection ~ 4500 2600
+Wire Wire Line
+	4500 2250 4500 2100
 $EndSCHEMATC

Commit message: updated the kicad project
Parts:
- BT1: symbol Battery -> Battery-RESCUE-sensor-node
Changed lines of the file:
@@
 EESchema Schematic File Version 2
+LIBS:sensor-node-rescue
 LIBS:power
 LIBS:device
@@
 $EndComp
 $Comp
-L Battery BT1
+L Battery-RESCUE-sensor-node BT1
 U 1 1 5877E2B9
 P 1100 3550
